File: buck.sch (EAGLE design)
At the start: 4 parts, among them U1 TPS54KC23RZRR

Commit message: added ldo schematic
Parts:
- removed R1_0805, R3_0805: (no value), rcl:R-US_R0805
- added J1: 163-179PH-EX, 163-179PH-EX:163-179PH-EX
Connections:
- removed net N$1: R1_0805.1, R3_0805.2
- removed net N$3: R3_0805.1, U1.EN
- new net N$2: J1.B, J1.C
- net VCC: now also J1.A; no longer R1_0805.2
Other:
- note added: "Battery Jack Connector 5.5x2.1mm"
Changed lines of the file:
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@@
 <part name="P+1" library="supply1" library_urn="urn:adsk.eagle:library:371" deviceset="VCC" device=""/>
 <part name="X_1" library="ngspice-simulation" library_urn="urn:adsk.eagle:library:527439" deviceset="GND" device=""/>
-<part name="R1_0805" library="rcl" library_urn="urn:adsk.eagle:library:334" deviceset="R-US_" device="R0805" package3d_urn="urn:adsk.eagle:package:23553/2"/>
 <part name="R2_0603" library="rcl" library_urn="urn:adsk.eagle:library:334" deviceset="R-US_" device="R0603" package3d_urn="urn:adsk.eagle:package:23555/3"/>
-<part name="R3_0805" library="rcl" library_urn="urn:adsk.eagle:library:334" deviceset="R-US_" device="R0805" package3d_urn="urn:adsk.eagle:package:23553/2"/>
-<part name="P+2" library="supply1" library_urn="urn:adsk.eagle:library:371" deviceset="VCC" device=""/>
 <part name="X_2" library="ngspice-simulation" library_urn="urn:adsk.eagle:library:527439" deviceset="GND" device=""/>
+<part name="J1" library="163-179PH-EX" deviceset="163-179PH-EX" device=""/>
 </parts>
 <sheets>
@@
 pins and as close as possible. minimizes parasistic
 impedance and lowers thermal resistance</text>
+<text x="-27.94" y="78.74" size="1.778" layer="91">Battery Jack Connector 5.5x2.1mm</text>
 </plain>
 <instances>
@@
 </instance>
 <instance part="X_1" gate="G$1" x="83.82" y="40.64" smashed="yes"/>
-<instance part="R1_0805" gate="G$1" x="17.78" y="86.36" smashed="yes" rot="R90">
-<attribute name="NAME" x="16.2814" y="82.55" size="1.778" layer="95" rot="R90"/>
-<attribute name="VALUE" x="21.082" y="82.55" size="1.778" layer="96" rot="R90"/>
-</instance>
 <instance part="R2_0603" gate="G$1" x="12.7" y="27.94" smashed="yes">
 <attribute name="NAME" x="8.89" y="29.4386" size="1.778" layer="95"/>
 <attribute name="VALUE" x="8.89" y="24.638" size="1.778" layer="96"/>
 </instance>
-<instance part="R3_0805" gate="G$1" x="17.78" y="73.66" smashed="yes" rot="R90">
-<attribute name="NAME" x="16.2814" y="69.85" size="1.778" layer="95" rot="R90"/>
-<attribute name="VALUE" x="21.082" y="69.85" size="1.778" layer="96" rot="R90"/>
+<instance part="X_2" gate="G$1" x="78.74" y="33.02" smashed="yes"/>
+<instance part="J1" gate="G$1" x="-22.86" y="86.36" smashed="yes">
+<attribute name="NAME" x="-6.35" y="93.98" size="1.778" layer="95" align="center-left"/>
+<attribute name="VALUE" x="-6.35" y="91.44" size="1.778" layer="96" align="center-left"/>
 </instance>
-<instance part="P+2" gate="VCC" x="17.78" y="96.52" smashed="yes">
-<attribute name="VALUE" x="15.24" y="93.98" size="1.778" layer="96" rot="R90"/>
-</instance>
-<instance part="X_2" gate="G$1" x="78.74" y="33.02" smashed="yes"/>
 </instances>
 <busses>
@@
 </segment>
 <segment>
-<pinref part="R1_0805" gate="G$1" pin="2"/>
-<wire x1="17.78" y1="91.44" x2="17.78" y2="93.98" width="0.1524" layer="91"/>
-<pinref part="P+2" gate="VCC" pin="VCC"/>
+<pinref part="J1" gate="G$1" pin="A"/>
+<wire x1="-2.54" y1="83.82" x2="2.54" y2="83.82" width="0.1524" layer="91"/>
+<label x="2.54" y="83.82" size="1.778" layer="95"/>
 </segment>
 </net>
@@
 </segment>
 </net>
-<net name="N$1" class="0">
+<net name="N$2" class="0">
 <segment>
-<pinref part="R1_0805" gate="G$1" pin="1"/>
-<pinref part="R3_0805" gate="G$1" pin="2"/>
-<wire x1="17.78" y1="81.28" x2="17.78" y2="78.74" width="0.1524" layer="91"/>
+<pinref part="J1" gate="G$1" pin="C"/>
+<wire x1="-2.54" y1="86.36" x2="2.54" y2="86.36" width="0.1524" layer="91"/>
+<wire x1="2.54" y1="86.36" x2="2.54" y2="91.44" width="0.1524" layer="91"/>
+<wire x1="2.54" y1="91.44" x2="-22.86" y2="91.44" width="0.1524" layer="91"/>
+<pinref part="J1" gate="G$1" pin="B"/>
+<wire x1="-22.86" y1="91.44" x2="-22.86" y2="86.36" width="0.1524" layer="91"/>
 </segment>
 </net>
-<net name="N$3" class="0">
-<segment>
-<pinref part="R3_0805" gate="G$1" pin="1"/>
-<wire x1="17.78" y1="68.58" x2="17.78" y2="66.04" width="0.1524" layer="91"/>
-<pinref part="U1" gate="A" pin="EN"/>
-<wire x1="17.78" y1="66.04" x2="33.02" y2="66.04" width="0.1524" layer="91"/>
-</segment>
-</net>

Commit message: Added a bunch of resistors
Parts:
- added R1, R2, R3, R4, R5: (no value), rcl:R-US_R0603
Changed lines of the file:
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@@
 <part name="X_2" library="ngspice-simulation" library_urn="urn:adsk.eagle:library:527439" deviceset="GND" device=""/>
 <part name="J1" library="163-179PH-EX" deviceset="163-179PH-EX" device=""/>
+<part name="R1" library="rcl" library_urn="urn:adsk.eagle:library:334" deviceset="R-US_" device="R0603" package3d_urn="urn:adsk.eagle:package:23555/3"/>
+<part name="R2" library="rcl" library_urn="urn:adsk.eagle:library:334" deviceset="R-US_" device="R0603" package3d_urn="urn:adsk.eagle:package:23555/3"/>
+<part name="R3" library="rcl" library_urn="urn:adsk.eagle:library:334" deviceset="R-US_" device="R0603" package3d_urn="urn:adsk.eagle:package:23555/3"/>
+<part name="R4" library="rcl" library_urn="urn:adsk.eagle:library:334" deviceset="R-US_" device="R0603" package3d_urn="urn:adsk.eagle:package:23555/3"/>
+<part name="R5" library="rcl" library_urn="urn:adsk.eagle:library:334" deviceset="R-US_" device="R0603" package3d_urn="urn:adsk.eagle:package:23555/3"/>
 </parts>
 <sheets>
@@
 <attribute name="VALUE" x="-6.35" y="91.44" size="1.778" layer="96" align="center-left"/>
 </instance>
+<instance part="R1" gate="G$1" x="2.54" y="43.18" smashed="yes">
+<attribute name="NAME" x="-1.27" y="44.6786" size="1.778" layer="95"/>
+<attribute name="VALUE" x="-1.27" y="39.878" size="1.778" layer="96"/>
+</instance>
+<instance part="R2" gate="G$1" x="2.54" y="38.1" smashed="yes">
+<attribute name="NAME" x="-1.27" y="39.5986" size="1.778" layer="95"/>
+<attribute name="VALUE" x="-1.27" y="34.798" size="1.778" layer="96"/>
+</instance>
+<instance part="R3" gate="G$1" x="-10.16" y="35.56" smashed="yes">
+<attribute name="NAME" x="-13.97" y="37.0586" size="1.778" layer="95"/>
+<attribute name="VALUE" x="-13.97" y="32.258" size="1.778" layer="96"/>
+</instance>
+<instance part="R4" gate="G$1" x="-12.7" y="43.18" smashed="yes">
+<attribute name="NAME" x="-16.51" y="44.6786" size="1.778" layer="95"/>
+<attribute name="VALUE" x="-16.51" y="39.878" size="1.778" layer="96"/>
+</instance>
+<instance part="R5" gate="G$1" x="2.54" y="55.88" smashed="yes">
+<attribute name="NAME" x="-1.27" y="57.3786" size="1.778" layer="95"/>
+<attribute name="VALUE" x="-1.27" y="52.578" size="1.778" layer="96"/>
+</instance>
 </instances>

Commit message: Deleted Felipe's Resistor
Parts:
- removed R4, R5: (no value), rcl:R-US_R0603
Changed lines of the file:
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@@
 <part name="R2" library="rcl" library_urn="urn:adsk.eagle:library:334" deviceset="R-US_" device="R0603" package3d_urn="urn:adsk.eagle:package:23555/3"/>
 <part name="R3" library="rcl" library_urn="urn:adsk.eagle:library:334" deviceset="R-US_" device="R0603" package3d_urn="urn:adsk.eagle:package:23555/3"/>
-<part name="R4" library="rcl" library_urn="urn:adsk.eagle:library:334" deviceset="R-US_" device="R0603" package3d_urn="urn:adsk.eagle:package:23555/3"/>
-<part name="R5" library="rcl" library_urn="urn:adsk.eagle:library:334" deviceset="R-US_" device="R0603" package3d_urn="urn:adsk.eagle:package:23555/3"/>
 </parts>
 <sheets>
@@
 <attribute name="VALUE" x="-13.97" y="32.258" size="1.778" layer="96"/>
 </instance>
-<instance part="R4" gate="G$1" x="-12.7" y="43.18" smashed="yes">
-<attribute name="NAME" x="-16.51" y="44.6786" size="1.778" layer="95"/>
-<attribute name="VALUE" x="-16.51" y="39.878" size="1.778" layer="96"/>
-</instance>
-<instance part="R5" gate="G$1" x="2.54" y="55.88" smashed="yes">
-<attribute name="NAME" x="-1.27" y="57.3786" size="1.778" layer="95"/>
-<attribute name="VALUE" x="-1.27" y="52.578" size="1.778" layer="96"/>
-</instance>
 </instances>

Commit message: Unified LDO, level shifter, and buck schematics. Using hierarchical circuit structure with modules abstracting more detailed subcircuits.
Connections:
- net VCC renamed VS_9V
Changed lines of the file:
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@@
 <parts>
 <part name="U1" library="TPS54KC23" deviceset="TPS54KC23RZRR" device=""/>
-<part name="P+1" library="supply1" library_urn="urn:adsk.eagle:library:371" deviceset="VCC" device=""/>
 <part name="X_1" library="ngspice-simulation" library_urn="urn:adsk.eagle:library:527439" deviceset="GND" device=""/>
 <part name="R2_0603" library="rcl" library_urn="urn:adsk.eagle:library:334" deviceset="R-US_" device="R0603" package3d_urn="urn:adsk.eagle:package:23555/3"/>
@@
 <attribute name="NAME" x="51.1556" y="82.7786" size="2.0828" layer="95" ratio="6" rot="SR0"/>
 <attribute name="VALUE" x="42.9006" y="80.2386" size="2.0828" layer="96" ratio="6" rot="SR0"/>
-</instance>
-<instance part="P+1" gate="VCC" x="27.94" y="83.82" smashed="yes">
-<attribute name="VALUE" x="25.4" y="81.28" size="1.778" layer="96" rot="R90"/>
 </instance>
 <instance part="X_1" gate="G$1" x="83.82" y="40.64" smashed="yes"/>
@@
 </busses>
 <nets>
-<net name="VCC" class="0">
-<segment>
-<pinref part="U1" gate="A" pin="VIN_2"/>
-<wire x1="33.02" y1="73.66" x2="27.94" y2="73.66" width="0.1524" layer="91"/>
-<wire x1="27.94" y1="73.66" x2="27.94" y2="81.28" width="0.1524" layer="91"/>
-<pinref part="P+1" gate="VCC" pin="VCC"/>
-<pinref part="U1" gate="A" pin="VIN"/>
-<wire x1="33.02" y1="71.12" x2="27.94" y2="71.12" width="0.1524" layer="91"/>
-<wire x1="27.94" y1="71.12" x2="27.94" y2="73.66" width="0.1524" layer="91"/>
-<junction x="27.94" y="73.66"/>
-</segment>
-<segment>
-<pinref part="J1" gate="G$1" pin="A"/>
-<wire x1="-2.54" y1="83.82" x2="2.54" y2="83.82" width="0.1524" layer="91"/>
-<label x="2.54" y="83.82" size="1.778" layer="95"/>
-</segment>
-</net>
 <net name="0" class="0">
 <segment>
@@
 </segment>
 </net>
+<net name="VS_9V" class="0">
+<segment>
+<pinref part="J1" gate="G$1" pin="A"/>
+<wire x1="-2.54" y1="83.82" x2="2.54" y2="83.82" width="0.1524" layer="91"/>
+<label x="2.54" y="83.82" size="1.778" layer="95"/>
+</segment>
+<segment>
+<pinref part="U1" gate="A" pin="VIN_2"/>
+<wire x1="33.02" y1="73.66" x2="27.94" y2="73.66" width="0.1524" layer="91"/>
+<wire x1="27.94" y1="73.66" x2="27.94" y2="81.28" width="0.1524" layer="91"/>
+<pinref part="U1" gate="A" pin="VIN"/>
+<wire x1="33.02" y1="71.12" x2="27.94" y2="71.12" width="0.1524" layer="91"/>
+<wire x1="27.94" y1="71.12" x2="27.94" y2="73.66" width="0.1524" layer="91"/>
+<junction x="27.94" y="73.66"/>
+<label x="24.638" y="82.042" size="1.778" layer="95"/>
+</segment>
+</net>
