File: system.sch (EAGLE design)
At the start: 6 parts, among them IC1 ATMEGA328P-MN, J1 163-179PH-EX, J2 TSW-104-07-F-S

Commit message: Fix some stuff
Connections:
- net V_1.25V renamed VS_1.5V
- net N$1: no longer IC1.IN+, R1.2
- net N$2: no longer IC1.OUT
- net N$4: now also IC1.IN+, R1.2
Changed lines of the file:
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@@
 <instances>
 <instance part="IC1" gate="G$1" x="33.02" y="30.48" smashed="yes">
-<attribute name="NAME" x="54.61" y="38.1" size="1.778" layer="95" align="center-left"/>
-<attribute name="VALUE" x="54.61" y="35.56" size="1.778" layer="96" align="center-left"/>
+<attribute name="NAME" x="39.37" y="38.1" size="1.778" layer="95" align="center-left"/>
+<attribute name="VALUE" x="39.37" y="35.56" size="1.778" layer="96" align="center-left"/>
 </instance>
 <instance part="R1" gate="G$1" x="7.62" y="25.4" smashed="yes">
@@
 <attribute name="VALUE" x="3.81" y="22.098" size="1.778" layer="96"/>
 </instance>
-<instance part="C1" gate="G$1" x="22.86" y="38.1" smashed="yes" rot="R90">
-<attribute name="NAME" x="22.225" y="39.116" size="1.778" layer="95" rot="R90"/>
-<attribute name="VALUE" x="27.051" y="39.116" size="1.778" layer="96" rot="R90"/>
+<instance part="C1" gate="G$1" x="17.78" y="33.02" smashed="yes">
+<attribute name="NAME" x="11.176" y="33.655" size="1.778" layer="95"/>
+<attribute name="VALUE" x="26.416" y="36.449" size="1.778" layer="96"/>
 </instance>
 <instance part="X_1" gate="G$1" x="22.86" y="17.78" smashed="yes"/>
@@
 <segment>
 <pinref part="IC1" gate="G$1" pin="V+"/>
-<wire x1="58.42" y1="27.94" x2="63.5" y2="27.94" width="0.1524" layer="91"/>
-<wire x1="63.5" y1="27.94" x2="63.5" y2="22.86" width="0.1524" layer="91"/>
-<label x="63.5" y="22.86" size="1.778" layer="95"/>
+<label x="71.12" y="27.94" size="1.778" layer="95"/>
+<wire x1="58.42" y1="27.94" x2="71.12" y2="27.94" width="0.1524" layer="91"/>
 </segment>
 </net>
-<net name="V_REF_1.15V" class="0">
+<net name="VS_BG" class="0">
 <segment>
 <wire x1="-10.16" y1="73.66" x2="7.62" y2="73.66" width="0.1524" layer="91"/>
 <label x="7.62" y="73.66" size="1.778" layer="95" xref="yes"/>
 <label x="-10.16" y="73.66" size="1.778" layer="95"/>
-</segment>
-</net>
-<net name="V_1.25V" class="0">
-<segment>
-<wire x1="-10.16" y1="66.04" x2="7.62" y2="66.04" width="0.1524" layer="91"/>
-<label x="7.62" y="66.04" size="1.778" layer="95" xref="yes"/>
-<label x="-10.16" y="66.04" size="1.778" layer="95"/>
-</segment>
-<segment>
-<pinref part="IC1" gate="G$1" pin="IN-"/>
-<wire x1="58.42" y1="30.48" x2="71.12" y2="30.48" width="0.1524" layer="91"/>
-<label x="71.12" y="30.48" size="1.778" layer="95"/>
 </segment>
 </net>
@@
 <label x="7.62" y="58.42" size="1.778" layer="95" xref="yes"/>
 <label x="-10.16" y="58.42" size="1.778" layer="95"/>
-</segment>
-</net>
-<net name="N$1" class="0">
-<segment>
-<pinref part="R1" gate="G$1" pin="2"/>
-<pinref part="IC1" gate="G$1" pin="IN+"/>
-<wire x1="12.7" y1="25.4" x2="15.24" y2="25.4" width="0.1524" layer="91"/>
-<wire x1="15.24" y1="25.4" x2="33.02" y2="25.4" width="0.1524" layer="91"/>
-<wire x1="15.24" y1="25.4" x2="15.24" y2="38.1" width="0.1524" layer="91"/>
-<junction x="15.24" y="25.4"/>
-<pinref part="C1" gate="G$1" pin="1"/>
-<wire x1="15.24" y1="38.1" x2="20.32" y2="38.1" width="0.1524" layer="91"/>
-</segment>
-</net>
-<net name="N$2" class="0">
-<segment>
-<pinref part="C1" gate="G$1" pin="2"/>
-<pinref part="IC1" gate="G$1" pin="OUT"/>
-<wire x1="27.94" y1="38.1" x2="33.02" y2="38.1" width="0.1524" layer="91"/>
-<wire x1="33.02" y1="38.1" x2="33.02" y2="30.48" width="0.1524" layer="91"/>
 </segment>
 </net>
@@
 </segment>
 </net>
+<net name="N$4" class="0">
+<segment>
+<wire x1="17.78" y1="38.1" x2="17.78" y2="35.56" width="0.1524" layer="91"/>
+<pinref part="C1" gate="G$1" pin="2"/>
+<pinref part="IC1" gate="G$1" pin="OUT"/>
+<wire x1="17.78" y1="38.1" x2="33.02" y2="38.1" width="0.1524" layer="91"/>
+<wire x1="33.02" y1="38.1" x2="33.02" y2="30.48" width="0.1524" layer="91"/>
+<pinref part="C1" gate="G$1" pin="1"/>
+<pinref part="IC1" gate="G$1" pin="IN+"/>
+<pinref part="R1" gate="G$1" pin="2"/>
+<wire x1="12.7" y1="25.4" x2="17.78" y2="25.4" width="0.1524" layer="91"/>
+<wire x1="17.78" y1="25.4" x2="33.02" y2="25.4" width="0.1524" layer="91"/>
+<wire x1="17.78" y1="27.94" x2="17.78" y2="25.4" width="0.1524" layer="91"/>
+<junction x="17.78" y="25.4"/>
+</segment>
+</net>
+<net name="VS_1.5V" class="0">
+<segment>
+<wire x1="-10.16" y1="66.04" x2="7.62" y2="66.04" width="0.1524" layer="91"/>
+<label x="7.62" y="66.04" size="1.778" layer="95" xref="yes"/>
+<label x="-10.16" y="66.04" size="1.778" layer="95"/>
+</segment>
+<segment>
+<pinref part="IC1" gate="G$1" pin="IN-"/>
+<wire x1="58.42" y1="30.48" x2="71.12" y2="30.48" width="0.1524" layer="91"/>
+<label x="71.12" y="30.48" size="1.778" layer="95"/>
+</segment>
+</net>

Commit message: added VS_1.5V ref in LDO schematic. cleaned up modules and changed atmega footprint.
Parts:
- removed IC1: ATMEGA328P-MN, ATMEGA328P-MN:ATMEGA328P-MN
- added U1: ATMEGA328PB-AU, ATMEGA328PB_AU32A:ATMEGA328PB-AU
Connections:
- removed net EN: IC1.EN
- removed net VS_1.5V: IC1.IN-
- removed net VS_2.5V: IC1.-IN, IC1.REF
- removed net V_SIG: IC1.+IN
- net 0: now also U1.GND_2; no longer IC1.-VS, IC1.EP, IC1.GND, IC1.GND_1, IC1.V-
- net N$1: no longer IC1.IN-, IC1.OUT, IC1.RT/CLK
- net N$2: no longer IC1.IN+, IC1.SW
- net N$3: no longer IC1.BST, IC1.IN-, IC1.OUTPUT
- net N$4: no longer IC1.IN+, IC1.IN-, IC1.OUT, IC1.RG_1, R1.2
- net N$5: no longer IC1.COMP, IC1.RG_2, R1.1
- net N$6: no longer IC1.FB
- net SCL: now also U1.(ADC5/PTCY/SCL0)PC5; no longer IC1.PC5_(ADC5/SCL/PCINT13)
- net SDA: now also U1.(ADC4/PTCY/SDA0)PC4; no longer IC1.PC4_(ADC4/SDA/PCINT12)
- net VS_5V: no longer IC1.+VS, IC1.V+
- net VS_6V: no longer IC1.V+
- net VS_9V: no longer IC1.VIN
- net V_BG: no longer IC1.IN+, IC1.OUT
Other:
- note added: "Non-inverting Amplifier Inputs: VS_5V, V_BG Outputs: VS_1.5V Vout = (1 + R5/R6)*Vin"
- note added: "to ATmega ADC"
- moved on the sheet: R1, R2

Commit message: Update ADC and MCU wiring
Finished ADC module
Wired ADC ports to MCU
Corrected amplification and filtering module
Connections:
- new net ADC_EXT_INT: U1.(PTCXY/INT0/OC3B/OC4B)PD2
- new net RST_ADC: U1.(ADC0/PTCY/MISO1)PC0
- new net V_TOGGLE: U1.(ADC1/PTCY/SCK1)PC1
Other:
- note added: "Instrumentation Amp with 500 gain"
- note added: "RST Logic: - When RST is high, S3A and D3 are shorted, allowing cap to discharge - When RST is low, S3B and D3 are shorted, and S3B is left open so there is no path for current to flow there. This is the regular state of the switch and reset occurs at end of every ADC measuring cycle"
- note added: "Second order sallen key filter with 20Hz cutoff, no gain"
- note added: "V_TOGGLE, RST_ADC, ADC_EXT_INT pins will need to be configured in the EICRA register of the MCU. - ADC_EXT_INT needs to be set to falling edge detection - V_TOGGLE needs to be a clock interrupt - RST_ADC needs to be high when Tin is saved into memory"
- note removed: "Instrumentation Amp with gain of 100"
- note removed: "Maybe do no gain and keep it a unity buffer?"
- note removed: "Second order Sallen-Key filter with 20Hz cutoff and gain of 5"

Commit message: cleaned up ports
Other:
- note added: "ADC_EXT_INT: ADC External Interrupt output of comparator, will go to MCU to trigger counting"
- note added: "PD2: input interrupt PC1: output interrupt PC0: output interrupt"
- moved on the sheet: R2

Commit message: adding MCU routing and values for R5 and R6 in LDO
Parts:
- added C1: 1uF, rcl:C-USC0603
- added C2: (no value), rcl:C-USC0603
Connections:
- new net VS_2.5V: C1.1, C2.1
- new net V_TP: C1.2
- net 0: now also C1.2, C2.2, U1.GND
- net N$2: now also C1.2
- net N$4: now also C1.1, C2.2
- net VS_5V: now also C1.1, C2.1, U1.AVCC, U1.VCC
- net VS_6V: now also C2.1
- net VS_9V: now also C1.1
- net V_BG: now also C1.1
Other:
- note added: "Comparator"
- note added: "Decoupling cap"
- note added: "TODO: add backup LDO"

Commit message: Added LDO, Changed switches for ADC, added 0 hm R's for power
Parts:
- added C3: 1uF, rcl:C-USC0603
- added C4, C5: 22uF, rcl:C-USC0603
- added IC1: TPS7B8650BQDDARQ1, TPS7B8650BQDDARQ1:TPS7B8650BQDDARQ1
- added R3, R4, R5, R6, R7: 0, rcl:R-US_R0603
Connections:
- new net EN: IC1.EN
- new net N$10: IC1.FB/NC, R6.1, R7.2
- new net N$9: C3.1, C5.1, IC1.EN, IC1.IN, R4.2
- new net VS_1.5V: C3.1, IC1.IN+, R5.2
- new net V_SIG: C3.2
- net 0: now also C3.2, C4.2, C5.2, IC1.-VS, IC1.EP, IC1.GND, IC1.V-, R4.1, R6.1, R7.1
- net N$1: now also IC1.IN-, IC1.OUT, IC1.RT/CLK, R3.2
- net N$2: now also C3.2, IC1.IN+, IC1.SW, R3.1, R3.2, R4.2; no longer C1.2
- net N$3: now also C1.2, C3.1, IC1.BST, IC1.IN-, IC1.OUT, IC1.OUTPUT, R3.1
- net N$4: now also IC1.IN-, IC1.OUT, IC1.RG_1, R3.1, R4.2
- net N$5: now also IC1.COMP, IC1.RG_2, R4.1, R5.2
- net N$6: now also C3.1, IC1.FB, R3.2, R5.1, R6.2
- net N$7: now also C4.1, C5.1, R3.1, R4.1, R5.1
- net VS_2.5V: now also IC1.-IN, IC1.REF
- net VS_5V: now also C4.1, IC1.+VS, IC1.OUT, IC1.V+, R3.2, R5.1, R5.2, R6.2, R7.1, R7.2
- net VS_6V: now also IC1.V+
- net VS_9V: now also IC1.VIN
- net V_BG: now also IC1.IN+, IC1.OUT, R3.2
- net V_TP: now also IC1.+IN
Other:
- note added: "RST Logic: - When RST is high, S2 and D are shorted, allowing cap to discharge - When RST is low, S1 and D are shorted, and S1 is left open so there is no path for current to flow there. This is the regular state of the switch and reset occurs at end of every ADC measuring cycle"
- note added: "V_TOGGLE = 1: V_SIG V_TOGGLE = 0: V_BG"
- note removed: "NOTE: Can delete and place 0 ohm resistors"
- note removed: "RST Logic: - When RST is high, S3A and D3 are shorted, allowing cap to discharge - When RST is low, S3B and D3 are shorted, and S3B is left open so there is no path for current to flow there. This is the regular state of the switch and reset occurs at end of every ADC measuring cycle"

Commit message: Updated R & C to correct model
Updated all Rs and Cs of ADC and amplifier to 0603
Added 0 ohm resistors to ADC power supply inputs and routed V_SIG to MCU ADC with a 0 ohm resistor
Parts:
- added R10, R11, R8, R9: 0, rcl:R-US_R0603
Connections:
- new net N$11: R8.1, U1.(ADC2/PTCY)PC2
- new net N$12: R9.2
- new net N$13: R10.2
- new net N$14: R11.1
- net ADC_EXT_INT: now also R11.2
- net N$3: now also R4.1, R8.1; no longer R3.1
- net N$4: now also R1.1; no longer R2.1
- net N$5: now also R1.2; no longer R2.2
- net N$6: now also R4.2; no longer C3.1, R3.2
- net N$7: now also R5.2; no longer C4.1, R1.2
- net VS_1.5V: now also R10.1
- net VS_2.5V: now also C5.1; no longer C1.1, C2.1
- net VS_5V: now also R8.2, R9.1
- net V_SIG: now also R8.2; no longer C3.2
- net V_TP: no longer C1.2
