File: system.brd (EAGLE design)
At the start: 160 x 100 mm, 125 parts, among them IC1 TPS7B8650BQDDARQ1, IC2 TLV9101IDBVR, IC3 TLV9101IDBVR, J1 TSW-104-07-F-S, J2 163-179PH-EX, J3 RS1-02-G, SW1 1825910-6, SW2 1825910-6, SW3 1825910-6, U1 ATMEGA328PB-AU

Commit message: Added EXT CLK
Added an external clock of 16MHz to MCU
Parts:
- added C10, C9: 22pF, rcl:C0603
- added Y1: ABL-16.000MHZ-B2, ABL-16.000MHZ-B2:ABL
Connections:
- new net EXT_CLK_1: C9.2, U1.7, Y1.1
- new net EXT_CLK_2: C10.2, U1.8, Y1.2
- net 0: now also C10.1, C9.1
Changed lines of the file:
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@@
 <attribute name="VALUE" x="-64.77" y="73.66" size="1.27" layer="27" ratio="6" rot="SR0"/>
+</element>
+<element name="Y1" library="ABL-16.000MHZ-B2" package="ABL" value="ABL-16.000MHZ-B2" x="-128.27" y="-3.81" smashed="yes">
+<attribute name="DESCRIPTION" value="ABRACON - ABL-16.000MHZ-B2 - CRYSTAL" x="-128.27" y="-3.81" size="1.778" layer="27" display="off"/>
+<attribute name="HEIGHT" value="mm" x="-128.27" y="-3.81" size="1.778" layer="27" display="off"/>
+<attribute name="MANUFACTURER_NAME" value="ABRACON" x="-128.27" y="-3.81" size="1.778" layer="27" display="off"/>
+<attribute name="MANUFACTURER_PART_NUMBER" value="ABL-16.000MHZ-B2" x="-128.27" y="-3.81" size="1.778" layer="27" display="off"/>
+<attribute name="MOUSER_PART_NUMBER" value="815-ABL-16-B2" x="-128.27" y="-3.81" size="1.778" layer="27" display="off"/>
+<attribute name="MOUSER_PRICE-STOCK" value="https://www.mouser.co.uk/ProductDetail/ABRACON/ABL-16.000MHZ-B2?qs=A7YjigRBFZlH19Ss3q%252BAbA%3D%3D" x="-128.27" y="-3.81" size="1.778" layer="27" display="off"/>
+<attribute name="NAME" x="-125.83" y="-3.81" size="1.27" layer="25" align="center"/>
+<attribute name="VALUE" x="-125.83" y="-3.81" size="1.27" layer="27" align="center"/>
+</element>
+<element name="C9" library="rcl" library_urn="urn:adsk.eagle:library:334" package="C0603" package3d_urn="urn:adsk.eagle:package:23616/2" value="22pF" x="-132.08" y="-10.16" smashed="yes">
+<attribute name="NAME" x="-132.715" y="-9.525" size="1.27" layer="25"/>
+<attribute name="POPULARITY" value="37" x="-132.08" y="-10.16" size="1.778" layer="27" display="off"/>
+<attribute name="SPICEPREFIX" value="C" x="-132.08" y="-10.16" size="1.778" layer="27" display="off"/>
+<attribute name="VALUE" x="-132.715" y="-12.065" size="1.27" layer="27"/>
+</element>
+<element name="C10" library="rcl" library_urn="urn:adsk.eagle:library:334" package="C0603" package3d_urn="urn:adsk.eagle:package:23616/2" value="22pF" x="-132.08" y="-13.97" smashed="yes">
+<attribute name="NAME" x="-132.715" y="-13.335" size="1.27" layer="25"/>
+<attribute name="POPULARITY" value="37" x="-132.08" y="-13.97" size="1.778" layer="27" display="off"/>
+<attribute name="SPICEPREFIX" value="C" x="-132.08" y="-13.97" size="1.778" layer="27" display="off"/>
+<attribute name="VALUE" x="-132.715" y="-15.875" size="1.27" layer="27"/>
 </element>
 </elements>
@@
 <contactref element="DUAL_SLOPE_ADC:C2" pad="2"/>
 <contactref element="DUAL_SLOPE_ADC:IC3" pad="2"/>
+<contactref element="C9" pad="1"/>
+<contactref element="C10" pad="1"/>
 <wire x1="-19.9" y1="210.82" x2="-21.57" y2="215.9" width="0" layer="19" extent="1-1"/>
 <wire x1="-16.93" y1="205.74" x2="-19.9" y2="210.82" width="0" layer="19" extent="1-1"/>
@@
 <wire x1="-85.51" y1="2.54" x2="-94.4" y2="36.83" width="0" layer="19" extent="1-1"/>
 <wire x1="-113.45" y1="2.54" x2="-85.51" y2="2.54" width="0" layer="19" extent="1-1"/>
+<wire x1="-132.93" y1="-10.16" x2="-113.45" y2="2.54" width="0" layer="19" extent="1-1"/>
+<wire x1="-132.93" y1="-13.97" x2="-132.93" y2="-10.16" width="0" layer="19" extent="1-1"/>
 </signal>
 <signal name="BATTERY_AND_BUCK:N$2">
@@
 <wire x1="-111.74" y1="187.64" x2="-44.47" y2="192.72" width="0" layer="19" extent="1-1"/>
 </signal>
+<signal name="EXT_CLK_1">
+<contactref element="C9" pad="2"/>
+<contactref element="Y1" pad="1"/>
+<contactref element="U1" pad="7"/>
+<wire x1="-128.27" y1="-3.81" x2="-131.23" y2="-10.16" width="0" layer="19" extent="1-1"/>
+<wire x1="-69.02" y1="71.66" x2="-128.27" y2="-3.81" width="0" layer="19" extent="1-1"/>
+</signal>
+<signal name="EXT_CLK_2">
+<contactref element="Y1" pad="2"/>
+<contactref element="C10" pad="2"/>
+<contactref element="U1" pad="8"/>
+<wire x1="-123.39" y1="-3.81" x2="-131.23" y2="-13.97" width="0" layer="19" extent="1-1"/>
+<wire x1="-69.02" y1="70.86" x2="-123.39" y2="-3.81" width="0" layer="19" extent="1-1"/>
+</signal>
 </signals>

Commit message: Moved ADC components to bottom right corner
Parts:
- moved DUAL_SLOPE_ADC:IC1 302.3 mm to (132.1, 6.35), turned to 180 degrees
- moved DUAL_SLOPE_ADC:IC5 278.7 mm to (147.3, 14.0)
- moved DUAL_SLOPE_ADC:R1 278.5 mm to (137.2, 7.62)
- moved DUAL_SLOPE_ADC:R2 271.7 mm to (113.0, 15.2), turned to 270 degrees
- moved DUAL_SLOPE_ADC:IC4 250.6 mm to (132.1, 15.2)
- moved DUAL_SLOPE_ADC:C2 246.1 mm to (121.9, 15.2)
- moved DUAL_SLOPE_ADC:C1 240.8 mm to (132.1, 11.4)
- moved DUAL_SLOPE_ADC:IC3 228.7 mm to (118.1, 12.7)
- moved IC3 27.4 mm to (-30.5, 190.5)
- moved U1 12.5 mm to (-53.3, 68.6)
- moved BATTERY_AND_BUCK:L1 6.35 mm to (-44.5, 87.6)
- moved SW2 2.84 mm to (-44.5, 177.8)
- moved SW1 2.84 mm to (-34.3, 177.8)
- moved SW3 2.84 mm to (-54.6, 177.8)

Commit message: added caps
Parts:
- added C11, C12, C13: 1uF, rcl:C0603
- AMP_AND_FILTER:R4, AMP_AND_FILTER:R5, DUAL_SLOPE_ADC:R2: value 10000 -> 10k
- BANDGAP_REF:R1: value 40000 -> 40k
- LDO_AND_VOLTAGE_REFS:R3, LDO_AND_VOLTAGE_REFS:R4, R7, R8, THERMISTOR_THERMOPILE:R1: value 2000000 -> 2M
- LDO_AND_VOLTAGE_REFS:R5: value 560000 -> 560k
- LDO_AND_VOLTAGE_REFS:R6: value 240000 -> 240k
- R24: value 100000 -> 100k
Connections:
- net 0: now also C11.2, C12.2, C13.2
- net VS_1.5V_OUT: now also C13.1
- net VS_2.5V_OUT: now also C12.1
- net VS_5V_OUT: now also C11.1

Commit message: update some stuff
Parts:
- removed LDO_AND_VOLTAGE_REFS:C3, LDO_AND_VOLTAGE_REFS:C5: 1uF, rcl:C0603
Connections:
- net 0: no longer LDO_AND_VOLTAGE_REFS:C3.2, LDO_AND_VOLTAGE_REFS:C5.2
- net VS_1.5V: no longer LDO_AND_VOLTAGE_REFS:C3.1
- net VS_2.5V: no longer LDO_AND_VOLTAGE_REFS:C5.1
Changed lines of the file:
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@@
 <attribute name="VALUE" x="-114.3" y="2.54" size="1.27" layer="27"/>
-</element>
-<element name="LDO_AND_VOLTAGE_REFS:C3" library="rcl" library_urn="urn:adsk.eagle:library:334" package="C0603" package3d_urn="urn:adsk.eagle:package:23616/2" value="1uF" x="-39.37" y="36.83" smashed="yes">
-<attribute name="NAME" x="-39.37" y="36.83" size="1.27" layer="25"/>
-<attribute name="POPULARITY" value="37" x="-39.37" y="36.83" size="1.778" layer="27" display="off"/>
-<attribute name="SPICEPREFIX" value="C" x="-39.37" y="36.83" size="1.778" layer="27" display="off"/>
-<attribute name="VALUE" x="-39.37" y="36.83" size="1.27" layer="27"/>
 </element>
 <element name="LDO_AND_VOLTAGE_REFS:C4" library="rcl" library_urn="urn:adsk.eagle:library:334" package="C0603" package3d_urn="urn:adsk.eagle:package:23616/2" value="1uF" x="-67.31" y="36.83" smashed="yes">
@@
 <attribute name="SPICEPREFIX" value="C" x="-67.31" y="36.83" size="1.778" layer="27" display="off"/>
 <attribute name="VALUE" x="-67.31" y="36.83" size="1.27" layer="27"/>
-</element>
-<element name="LDO_AND_VOLTAGE_REFS:C5" library="rcl" library_urn="urn:adsk.eagle:library:334" package="C0603" package3d_urn="urn:adsk.eagle:package:23616/2" value="1uF" x="-95.25" y="36.83" smashed="yes">
-<attribute name="NAME" x="-95.25" y="36.83" size="1.27" layer="25"/>
-<attribute name="POPULARITY" value="37" x="-95.25" y="36.83" size="1.778" layer="27" display="off"/>
-<attribute name="SPICEPREFIX" value="C" x="-95.25" y="36.83" size="1.778" layer="27" display="off"/>
-<attribute name="VALUE" x="-95.25" y="36.83" size="1.27" layer="27"/>
 </element>
 <element name="LDO_AND_VOLTAGE_REFS:IC1" library="TLV9101IDBVR" package="SOT95P280X145-5N" value="TLV9101IDBVR" x="-111.76" y="46.99" smashed="yes">
@@
 <contactref element="LDO_AND_VOLTAGE_REFS:IC3" pad="4"/>
 <contactref element="LDO_AND_VOLTAGE_REFS:IC3" pad="1"/>
-<contactref element="LDO_AND_VOLTAGE_REFS:C3" pad="1"/>
 <wire x1="-58.4" y1="53.02" x2="-104.99" y2="205.74" width="0" layer="19" extent="1-1"/>
 <wire x1="-55.9" y1="51.12" x2="-58.4" y2="53.02" width="0" layer="19" extent="1-1"/>
-<wire x1="-40.22" y1="36.83" x2="-55.9" y2="51.12" width="0" layer="19" extent="1-1"/>
 </signal>
 <signal name="VS_2.5V">
@@
 <contactref element="LDO_AND_VOLTAGE_REFS:IC2" pad="1"/>
 <contactref element="LDO_AND_VOLTAGE_REFS:IC2" pad="4"/>
-<contactref element="LDO_AND_VOLTAGE_REFS:C5" pad="1"/>
 <wire x1="-29.19" y1="53.02" x2="-49.11" y2="205.74" width="0" layer="19" extent="1-1"/>
 <wire x1="-26.69" y1="51.12" x2="-29.19" y2="53.02" width="0" layer="19" extent="1-1"/>
-<wire x1="-96.1" y1="36.83" x2="-29.19" y2="53.02" width="0" layer="19" extent="1-1"/>
 </signal>
 <signal name="ADC_EXT_INT">
@@
 <contactref element="BATTERY_AND_BUCK:C5" pad="2"/>
 <contactref element="BATTERY_AND_BUCK:C6" pad="2"/>
-<contactref element="LDO_AND_VOLTAGE_REFS:C5" pad="2"/>
 <contactref element="LDO_AND_VOLTAGE_REFS:IC3" pad="2"/>
 <contactref element="LDO_AND_VOLTAGE_REFS:IC1" pad="2"/>
@@
 <contactref element="LDO_AND_VOLTAGE_REFS:IC2" pad="2"/>
 <contactref element="LDO_AND_VOLTAGE_REFS:J1" pad="2"/>
-<contactref element="LDO_AND_VOLTAGE_REFS:C3" pad="2"/>
 <contactref element="LDO_AND_VOLTAGE_REFS:R6" pad="1"/>
 <contactref element="BANDGAP_REF:Q1" pad="5"/>
@@
 <wire x1="-40.22" y1="46.99" x2="-29.19" y2="52.07" width="0" layer="19" extent="1-1"/>
 <wire x1="-40.22" y1="41.91" x2="-40.22" y2="46.99" width="0" layer="19" extent="1-1"/>
-<wire x1="-38.52" y1="36.83" x2="-40.22" y2="41.91" width="0" layer="19" extent="1-1"/>
-<wire x1="-35.56" y1="20.32" x2="-38.52" y2="36.83" width="0" layer="19" extent="1-1"/>
 <wire x1="-58.4" y1="52.07" x2="-40.22" y2="46.99" width="0" layer="19" extent="1-1"/>
 <wire x1="-57.59" y1="68.18" x2="-58.4" y2="52.07" width="0" layer="19" extent="1-1"/>
 <wire x1="-49.09" y1="68.98" x2="-57.59" y2="68.18" width="0" layer="19" extent="1-1"/>
 <wire x1="-66.46" y1="36.83" x2="-58.4" y2="52.07" width="0" layer="19" extent="1-1"/>
+<wire x1="-35.56" y1="20.32" x2="-40.22" y2="41.91" width="0" layer="19" extent="1-1"/>
 <wire x1="-131.23" y1="102.87" x2="-107.1" y2="102.87" width="0" layer="19" extent="1-1"/>
 <wire x1="-132.93" y1="90.17" x2="-131.23" y2="102.87" width="0" layer="19" extent="1-1"/>
-<wire x1="-94.4" y1="36.83" x2="-66.46" y2="36.83" width="0" layer="19" extent="1-1"/>
-<wire x1="-96.1" y1="41.91" x2="-94.4" y2="36.83" width="0" layer="19" extent="1-1"/>
-<wire x1="-113.01" y1="46.99" x2="-96.1" y2="41.91" width="0" layer="19" extent="1-1"/>
 <wire x1="-99.48" y1="161.29" x2="-70.27" y2="161.29" width="0" layer="19" extent="1-1"/>
 <wire x1="-128.69" y1="161.29" x2="-99.48" y2="161.29" width="0" layer="19" extent="1-1"/>
-<wire x1="-85.51" y1="2.54" x2="-94.4" y2="36.83" width="0" layer="19" extent="1-1"/>
-<wire x1="-113.45" y1="2.54" x2="-85.51" y2="2.54" width="0" layer="19" extent="1-1"/>
-<wire x1="-132.93" y1="-10.16" x2="-113.45" y2="2.54" width="0" layer="19" extent="1-1"/>
-<wire x1="-132.93" y1="-13.97" x2="-132.93" y2="-10.16" width="0" layer="19" extent="1-1"/>
-<wire x1="-131.23" y1="-19.05" x2="-132.93" y2="-13.97" width="0" layer="19" extent="1-1"/>
-<wire x1="-131.23" y1="-24.13" x2="-131.23" y2="-19.05" width="0" layer="19" extent="1-1"/>
-<wire x1="-131.23" y1="-29.21" x2="-131.23" y2="-24.13" width="0" layer="19" extent="1-1"/>
+<wire x1="-96.1" y1="41.91" x2="-66.46" y2="36.83" width="0" layer="19" extent="1-1"/>
+<wire x1="-113.01" y1="46.99" x2="-96.1" y2="41.91" width="0" layer="19" extent="1-1"/>
 <wire x1="-101.18" y1="196.85" x2="-99.48" y2="161.29" width="0" layer="19" extent="1-1"/>
 <wire x1="-108.37" y1="205.74" x2="-101.18" y2="196.85" width="0" layer="19" extent="1-1"/>
@@
 <wire x1="-123.17" y1="210.82" x2="-123.61" y2="205.74" width="0" layer="19" extent="1-1"/>
 <wire x1="-114.72" y1="196.85" x2="-113.45" y2="205.74" width="0" layer="19" extent="1-1"/>
+<wire x1="-85.51" y1="2.54" x2="-66.46" y2="36.83" width="0" layer="19" extent="1-1"/>
+<wire x1="-113.45" y1="2.54" x2="-85.51" y2="2.54" width="0" layer="19" extent="1-1"/>
+<wire x1="-132.93" y1="-10.16" x2="-113.45" y2="2.54" width="0" layer="19" extent="1-1"/>
+<wire x1="-132.93" y1="-13.97" x2="-132.93" y2="-10.16" width="0" layer="19" extent="1-1"/>
+<wire x1="-131.23" y1="-19.05" x2="-132.93" y2="-13.97" width="0" layer="19" extent="1-1"/>
+<wire x1="-131.23" y1="-24.13" x2="-131.23" y2="-19.05" width="0" layer="19" extent="1-1"/>
+<wire x1="-131.23" y1="-29.21" x2="-131.23" y2="-24.13" width="0" layer="19" extent="1-1"/>
 <wire x1="116.86" y1="12.7" x2="-29.19" y2="52.07" width="0" layer="19" extent="1-1"/>
 <wire x1="122.77" y1="15.24" x2="116.86" y2="12.7" width="0" layer="19" extent="1-1"/>
